Commit message: test_gazebo_robot_model三轮小车模型

File: test_gazebo_robot_model/urdf/my_move_robot.xacro (robot description, xacro)
@@ -18,7 +18,7 @@
 		<visual>
 			<geometry>
-				<box size="0.001 0.001 0.001"/>
+				<cylinder length=".01" radius="0.117"/>
 			</geometry>
-			<origin rpy="0 0 0" xyz="0 0 0"/>
+			<origin rpy="0 0 1.57075" xyz="0 0 0"/>
 		</visual>
 		<xacro:default_inertial mass="0.0001"/>
@@ -32,7 +32,7 @@
 		<visual>
 			<geometry>
-				<box size="0.2 .3 .1"/>
+				<cylinder length="0.001" radius="0.001"/>
 			</geometry>
-			<origin rpy="0 0 1.54" xyz="0 0 0.05"/>
+			<origin rpy="0 0 1.57075" xyz="0 0 0"/>
 			<material name="white">
 				<color rgba="1 1 1 1"/>
@@ -41,5 +41,5 @@
 		<collision>
 			<geometry>
-				<box size="0.2 .3 0.1"/>
+				<cylinder length="0.001" radius="0.001"/>
 			</geometry>
 		</collision>
@@ -49,8 +49,8 @@
 		<visual>
 			<geometry>
-				<cylinder length="${length_wheel}" radius="${radius_wheel}"/>
+				<cylinder length=".02" radius="0.029"/>
 			</geometry>
 			<!-- <origin rpy="0 1.5 0" xyz="0.1 0.1 0"/> -->
-			<origin rpy="0 0 0" xyz="0 0 0"/>
+			<origin rpy="0 0 1.57075" xyz="0 0 0"/>
 			<material name="black">
 				<color rgba="0 0 0 1"/>
@@ -59,5 +59,5 @@
 		<collision>
 			<geometry>
-				<cylinder length="${length_wheel}" radius="${radius_wheel}"/>
+				<cylinder length=".02" radius="0.029"/>
 			</geometry>
 		</collision>
@@ -67,13 +67,13 @@
 		<visual>
 			<geometry>
-				<cylinder length="${length_wheel}" radius="${radius_wheel}"/>
+				<cylinder length=".02" radius="0.029"/>
 			</geometry>
 			<!-- <origin rpy="0 1.5 0" xyz="-0.1 0.1 0"/> -->
-			<origin rpy="0 0 0" xyz="0 0 0"/>
+			<origin rpy="0 0 1.57075" xyz="0 0 0"/>
 			<material name="black"/>
 		</visual>
 		<collision>
 			<geometry>
-				<cylinder length="${length_wheel}" radius="${radius_wheel}"/>
+				<cylinder length=".02" radius="0.029"/>
 			</geometry>
 		</collision>
@@ -83,13 +83,13 @@
 		<visual>
 			<geometry>
-				<cylinder length="${length_wheel}" radius="${radius_wheel}"/>
+				<cylinder length=".02" radius="0.029"/>
 			</geometry>
 			<!-- <origin rpy="0 1.5 0" xyz="0.1 -0.1 0"/> -->
-			<origin rpy="0 0 0" xyz="0 0 0"/>
+			<origin rpy="0 0 1.57075" xyz="0 0 0"/>
 			<material name="black"/>
 		</visual>
 		<collision>
 			<geometry>
-				<cylinder length="${length_wheel}" radius="${radius_wheel}"/>
+				<cylinder length=".02" radius="0.029"/>
 			</geometry>
 		</collision>
@@ -99,5 +99,5 @@
 		<visual>
 			<geometry>
-				<cylinder length="${length_wheel}" radius="${radius_wheel}"/>
+				<cylinder length="0.00001" radius="0.00001"/>
 			</geometry>
 			<!--    <origin rpy="0 1.5 0" xyz="-0.1 -0.1 0"/> -->
@@ -115,5 +115,5 @@
 		<parent link="base_link"/>
 		<child link="wheel_1"/>
-		<origin rpy="1.5707 0 0" xyz="0.1 0.15 0"/>
+		<origin rpy="1.57075 1.57075 0" xyz="0.117 0 -0.024"/>
 		<axis xyz="0 0 1" />
 	</joint>
@@ -124,5 +124,5 @@
 		<parent link="base_link"/>
 		<child link="wheel_2"/>
-		<origin rpy="1.5707 0 0" xyz="-0.1 0.15 0"/>
+		<origin rpy="1.57075 1.57075 0" xyz="-0.0585 0.1013 -0.024"/>
 	</joint>
 	<joint name="base_to_wheel3" type="continuous">
@@ -130,5 +130,5 @@
 		<axis xyz="0 0 1" />
 		<child link="wheel_3"/>
-		<origin rpy="1.5707 0 0" xyz="0.1 -0.15 0"/>
+		<origin rpy="1.57075 1.57075 0" xyz="-0.0585 -0.1013 -0.024"/>
 	</joint>
 	<joint name="base_to_wheel4" type="continuous">

Commit message: move_robot.xacro机器人模型模拟gazebo

File: test_gazebo_robot_model/urdf/my_move_robot.xacro (robot description, xacro)
@@ -5,6 +5,7 @@
 		xmlns:interface="http://playerstage.sourceforge.net/gazebo/xmlschema/#interface"
 		name="robot1_xacro">
-	<xacro:property name="length_wheel" value="0.05" />
-	<xacro:property name="radius_wheel" value="0.05" />
+	<property name="M_PI" value="3.1415926535897931"/>
+	<property name="base_radius" value="0.117" />
+	<property name="cube_2" value="1.414213562" />
 	<xacro:macro name="default_inertial" params="mass">
 		<inertial>
@@ -15,36 +16,5 @@
 		</inertial>
 	</xacro:macro>
-	<link name="base_footprint">
-		<visual>
-			<geometry>
-				<cylinder length=".01" radius="0.117"/>
-			</geometry>
-			<origin rpy="0 0 1.57075" xyz="0 0 0"/>
-		</visual>
-		<xacro:default_inertial mass="0.0001"/>
-	</link>
-	<joint name="base_footprint_joint" type="fixed">
-		<origin xyz="0 0 0" />
-		<parent link="base_footprint" />
-		<child link="base_link" />
-	</joint>
-	<link name="base_link">
-		<visual>
-			<geometry>
-				<cylinder length="0.001" radius="0.001"/>
-			</geometry>
-			<origin rpy="0 0 1.57075" xyz="0 0 0"/>
-			<material name="white">
-				<color rgba="1 1 1 1"/>
-			</material>
-		</visual>
-		<collision>
-			<geometry>
-				<cylinder length="0.001" radius="0.001"/>
-			</geometry>
-		</collision>
-		<xacro:default_inertial mass="10"/>
-	</link>
-	<link name="wheel_1">
+	<xacro:macro name="default_wheel">
 		<visual>
 			<geometry>
@@ -62,79 +32,72 @@
 			</geometry>
 		</collision>
-		<xacro:default_inertial mass="1"/>
-	</link>
-	<link name="wheel_2">
+	</xacro:macro>
+	<xacro:macro name="default_base_link">
 		<visual>
 			<geometry>
-				<cylinder length=".02" radius="0.029"/>
+				<cylinder length=".01" radius="${base_radius}"/>
 			</geometry>
-			<!-- <origin rpy="0 1.5 0" xyz="-0.1 0.1 0"/> -->
 			<origin rpy="0 0 1.57075" xyz="0 0 0"/>
-			<material name="black"/>
+			<material name="white">
+				<color rgba="1 1 1 1"/>
+			</material>
 		</visual>
 		<collision>
 			<geometry>
-				<cylinder length=".02" radius="0.029"/>
+				<cylinder length=".01" radius="${base_radius}"/>
 			</geometry>
 		</collision>
-		<xacro:default_inertial mass="1"/>
+	</xacro:macro>
+	<link name="base_link">
+		<xacro:default_base_link />
+		<xacro:default_inertial mass="10"/>
 	</link>
-	<link name="wheel_3">
-		<visual>
-			<geometry>
-				<cylinder length=".02" radius="0.029"/>
-			</geometry>
-			<!-- <origin rpy="0 1.5 0" xyz="0.1 -0.1 0"/> -->
-			<origin rpy="0 0 1.57075" xyz="0 0 0"/>
-			<material name="black"/>
-		</visual>
-		<collision>
-			<geometry>
-				<cylinder length=".02" radius="0.029"/>
-			</geometry>
-		</collision>
-		<xacro:default_inertial mass="1"/>
+	<link name="right_front_wheel">
+		<xacro:default_wheel />
+		<xacro:default_inertial mass="0.01"/>
 	</link>
-	<link name="wheel_4">
-		<visual>
-			<geometry>
-				<cylinder length="0.00001" radius="0.00001"/>
-			</geometry>
-			<!--    <origin rpy="0 1.5 0" xyz="-0.1 -0.1 0"/> -->
-			<origin rpy="0 0 0" xyz="0 0 0" />
-			<material name="black"/>
-		</visual>
-		<collision>
-			<geometry>
-				<cylinder length="${length_wheel}" radius="${radius_wheel}"/>
-			</geometry>
-		</collision>
-		<xacro:default_inertial mass="1"/>
+	<link name="right_back_wheel">
+		<xacro:default_wheel />
+		<xacro:default_inertial mass="0.01"/>
 	</link>
-	<joint name="base_to_wheel1" type="continuous">
+	<link name="left_front_wheel">
+		<xacro:default_wheel />
+		<xacro:default_inertial mass="0.01"/>
+	</link>
+	<link name="left_back_wheel">
+		<xacro:default_wheel />
+		<xacro:default_inertial mass="0.01"/>
+	</link>
+	<joint name="right_front_wheel_joint" type="continuous">
 		<parent link="base_link"/>
-		<child link="wheel_1"/>
-		<origin rpy="1.57075 1.57075 0" xyz="0.117 0 -0.024"/>
+		<child link="right_front_wheel"/>
+		<origin rpy="0 ${M_PI/2} 0" xyz="${base_radius/cube_2} ${base_radius/cube_2} -0.024"/>
 		<axis xyz="0 0 1" />
+		<limit effort="100" velocity="100"/>
+		<joint_properties damping="0.0" friction="0.0"/>
 	</joint>
-	<joint name="base_to_wheel2" type="continuous">
+	<joint name="right_back_wheel_joint" type="continuous">
 		<axis xyz="0 0 1" />
-		<anchor xyz="0 0 0" />
-		<limit effort="100" velocity="100" />
 		<parent link="base_link"/>
-		<child link="wheel_2"/>
-		<origin rpy="1.57075 1.57075 0" xyz="-0.0585 0.1013 -0.024"/>
+		<child link="right_back_wheel"/>
+		<origin rpy="0 ${M_PI/2} 0" xyz="${base_radius/cube_2} ${-base_radius/cube_2} -0.024"/>
+		<limit effort="100" velocity="100"/>
+		<joint_properties damping="0.0" friction="0.0"/>
 	</joint>
-	<joint name="base_to_wheel3" type="continuous">
+	<joint name="left_front_wheel_joint" type="continuous">
 		<parent link="base_link"/>
 		<axis xyz="0 0 1" />
-		<child link="wheel_3"/>
-		<origin rpy="1.57075 1.57075 0" xyz="-0.0585 -0.1013 -0.024"/>
+		<child link="left_front_wheel"/>
+		<origin rpy="0 ${M_PI/2} 0" xyz="${-base_radius/cube_2} ${base_radius/cube_2} -0.024"/>
+		<limit effort="100" velocity="100"/>
+		<joint_properties damping="0.0" friction="0.0"/>
 	</joint>
-	<joint name="base_to_wheel4" type="continuous">
+	<joint name="left_back_wheel_joint" type="continuous">
 		<parent link="base_link"/>
 		<axis xyz="0 0 1" />
-		<child link="wheel_4"/>
-		<origin rpy="1.5707 0 0" xyz="-0.1 -0.15 0"/>
+		<child link="left_back_wheel"/>
+		<origin rpy="0 ${M_PI/2} 0" xyz="${-base_radius/cube_2} ${-base_radius/cube_2} -0.024"/>
+		<limit effort="100" velocity="100"/>
+		<joint_properties damping="0.0" friction="0.0"/>
 	</joint>
 	<!-- Drive controller -->
@@ -143,13 +106,13 @@
 	    <updateRate>100.0</updateRate>
 	    <robotNamespace></robotNamespace>
-	    <leftFrontJoint>base_to_wheel1</leftFrontJoint>
-	    <rightFrontJoint>base_to_wheel3</rightFrontJoint>
-	    <leftRearJoint>base_to_wheel2</leftRearJoint>
-	    <rightRearJoint>base_to_wheel4</rightRearJoint>
+	    <leftFrontJoint>left_front_wheel_joint</leftFrontJoint>
+	    <rightFrontJoint>right_front_wheel_joint</rightFrontJoint>
+	    <leftRearJoint>left_back_wheel_joint</leftRearJoint>
+	    <rightRearJoint>right_back_wheel_joint</rightRearJoint>
 	    <wheelSeparation>4</wheelSeparation>
 	    <wheelDiameter>0.1</wheelDiameter>
 	    <commandTopic>cmd_vel</commandTopic>
 	    <odometryTopic>odom</odometryTopic>
-	    <robotBaseFrame>base_footprint</robotBaseFrame>
+	    <robotBaseFrame>base_link</robotBaseFrame>
 	    <odometryFrame>odom</odometryFrame>
 	    <torque>1</torque>

File: tmrobot_description/urdf/tmrobot.all.urdf.xacro (robot description, xacro)
@@ -1,127 +1,104 @@
 <?xml version="1.0"?>
-<robot name="table"
-    xmlns:xi="http://www.w3.org/2001/XInclude"
-    xmlns:gazebo="http://playerstage.sourceforge.net/gazebo/xmlschema/#gz"
-    xmlns:model="http://playerstage.sourceforge.net/gazebo/xmlschema/#model"
+<robot xmlns:xacro="http://www.ros.org/wiki/xacro"
     xmlns:sensor="http://playerstage.sourceforge.net/gazebo/xmlschema/#sensor"
-    xmlns:body="http://playerstage.sourceforge.net/gazebo/xmlschema/#body"
-    xmlns:geom="http://playerstage.sourceforge.net/gazebo/xmlschema/#geom"
-    xmlns:joint="http://playerstage.sourceforge.net/gazebo/xmlschema/#joint"
     xmlns:controller="http://playerstage.sourceforge.net/gazebo/xmlschema/#controller"
     xmlns:interface="http://playerstage.sourceforge.net/gazebo/xmlschema/#interface"
-    xmlns:rendering="http://playerstage.sourceforge.net/gazebo/xmlschema/#rendering"
-    xmlns:renderable="http://playerstage.sourceforge.net/gazebo/xmlschema/#renderable"
-    xmlns:physics="http://playerstage.sourceforge.net/gazebo/xmlschema/#physics"
-    xmlns:xacro="http://ros.org/wiki/xacro">
-    <property name="M_PI" value="3.1415926535897931"/>
-    <link name="base_link">
-      <inertial>
-        <mass value="1.0" />
-        <origin rpy="0 0 1.57075" xyz="0 0 0"/>
-        <inertia ixx="1" ixy="0"  ixz="0"
-                 iyy="1" iyz="0"
-                 izz="1" />
-      </inertial>
-      <visual>
-        <geometry>
-          <cylinder length=".01" radius="0.117"/>
-        </geometry>
-        <origin rpy="0 0 1.57075" xyz="0 0 0"/>
-        <material name="blue">
-          <color rgba="1 1 1 1"/>
-        </material>
-      </visual>
-    </link>
-    <joint name="front_wheel_joint" type="continuous">
-      <axis xyz="0 0 1"/>
-      <parent link="base_link"/>
-      <child link="front_wheel"/>
-      <origin rpy="1.57075 1.57075 0" xyz="0.117 0 -0.024"/>
-      <joint_properties damping="0.0" friction="0.0"/>
-    </joint>
-    <link name="front_wheel">
-      <inertial>
-        <mass value="1.0" />
-        <origin rpy="0 0 1.57075" xyz="0 0 0"/>
-        <inertia ixx="1" ixy="0"  ixz="0"
-                 iyy="1" iyz="0"
-                 izz="1" />
-      </inertial>
-      <visual>
-        <geometry>
-          <cylinder length=".02" radius="0.029"/>
-        </geometry>
-        <origin rpy="0 0 1.57075" xyz="0 0 0"/>
-        <material name="black">
-          <color rgba="0 0 0 1"/>
-        </material>
-      </visual>
-    </link>
-    <joint name="behind_left_wheel_joint" type="continuous">
-      <axis xyz="0 0 1"/>
-      <parent link="base_link"/>
-      <child link="behind_left_wheel"/>
-      <origin rpy="1.57075 1.57075 0" xyz="-0.0585 0.1013 -0.024"/>
-      <joint_properties damping="0.0" friction="0.0"/>
-    </joint>
-    <link name="behind_left_wheel">
-      <inertial>
-        <mass value="1.0" />
-        <origin rpy="0 0 1.57075" xyz="0 0 0"/>
-        <inertia ixx="1" ixy="0"  ixz="0"
-                 iyy="1" iyz="0"
-                 izz="1" />
-      </inertial>
-      <visual>
-        <geometry>
-          <cylinder length=".02" radius="0.029"/>
-        </geometry>
-        <origin rpy="0 0 1.57075" xyz="0 0 0"/>
-        <material name="black">
-          <color rgba="0 0 0 1"/>
-        </material>
-      </visual>
-    </link>
-    <joint name="behind_right_wheel_joint" type="continuous">
-      <axis xyz="0 0 1"/>
-      <parent link="base_link"/>
-      <child link="behind_right_wheel"/>
-      <origin rpy="1.57075 1.57075 0" xyz="-0.0585 -0.1013 -0.024"/>
-      <joint_properties damping="0.0" friction="0.0"/>
-    </joint>
-    <link name="behind_right_wheel">
-      <inertial>
-        <mass value="1.0" />
-        <origin rpy="0 0 1.57075" xyz="0 0 0"/>
-        <inertia ixx="1" ixy="0"  ixz="0"
-                 iyy="1" iyz="0"
-                 izz="1" />
-      </inertial>
-      <visual>
-        <geometry>
-          <cylinder length=".02" radius="0.029"/>
-        </geometry>
-        <origin rpy="0 0 1.57075" xyz="0 0 0"/>
-        <material name="black">
-          <color rgba="0 0 0 1"/>
-        </material>
-      </visual>
-    </link>
-    <gazebo reference="base_link">
-        <material>Gazebo/Blue</material>
-    </gazebo>
-    <gazebo reference="front_wheel">
-        <material>Gazebo/FlatBlack</material>
-    </gazebo>
-    <gazebo reference="behind_left_wheel">
-        <material>Gazebo/FlatBlack</material>
-    </gazebo>
-    <gazebo reference="behind_right_wheel">
-        <material>Gazebo/FlatBlack</material>
-    </gazebo>
-  <gazebo>
-    <static>true</static>
-    <canonicalBody>base_link</canonicalBody>
-  </gazebo>
+    name="robot1_xacro">
+  <property name="M_PI" value="3.1415926535897931"/>
+  <property name="base_radius" value="0.117" />
+  <property name="cube_2" value="1.414213562" />
+  <xacro:macro name="default_inertial" params="mass">
+    <inertial>
+    <mass value="${mass}" />
+    <inertia ixx="1.0" ixy="0.0" ixz="0.0"
+        iyy="1.0" iyz="0.0"
+        izz="1.0" />
+    </inertial>
+  </xacro:macro>
+  <xacro:macro name="default_wheel">
+    <visual>
+      <geometry>
+        <cylinder length=".02" radius="0.029"/>
+      </geometry>
+      <!-- <origin rpy="0 1.5 0" xyz="0.1 0.1 0"/> -->
+      <origin rpy="0 0 1.57075" xyz="0 0 0"/>
+      <material name="black">
+        <color rgba="0 0 0 1"/>
+      </material>
+    </visual>
+    <collision>
+      <geometry>
+        <cylinder length=".02" radius="0.029"/>
+      </geometry>
+    </collision>
+  </xacro:macro>
+  <xacro:macro name="default_base_link">
+    <visual>
+      <geometry>
+        <cylinder length=".01" radius="${base_radius}"/>
+      </geometry>
+      <origin rpy="0 0 1.57075" xyz="0 0 0"/>
+      <material name="white">
+        <color rgba="1 1 1 1"/>
+      </material>
+    </visual>
+    <collision>
+      <geometry>
+        <cylinder length=".01" radius="${base_radius}"/>
+      </geometry>
+    </collision>
+  </xacro:macro>
+  <link name="base_link">
+    <xacro:default_base_link />
+    <xacro:default_inertial mass="10"/>
+  </link>
+  <link name="right_front_wheel">
+    <xacro:default_wheel />
+    <xacro:default_inertial mass="0.01"/>
+  </link>
+  <link name="right_back_wheel">
+    <xacro:default_wheel />
+    <xacro:default_inertial mass="0.01"/>
+  </link>
+  <link name="left_front_wheel">
+    <xacro:default_wheel />
+    <xacro:default_inertial mass="0.01"/>
+  </link>
+  <link name="left_back_wheel">
+    <xacro:default_wheel />
+    <xacro:default_inertial mass="0.01"/>
+  </link>
+  <joint name="right_front_wheel_joint" type="continuous">
+    <parent link="base_link"/>
+    <child link="right_front_wheel"/>
+    <origin rpy="0 ${M_PI/2} 0" xyz="${base_radius/cube_2} ${base_radius/cube_2} -0.024"/>
+    <axis xyz="0 0 1" />
+    <limit effort="100" velocity="100"/>
+    <joint_properties damping="0.0" friction="0.0"/>
+  </joint>
+  <joint name="right_back_wheel_joint" type="continuous">
+    <axis xyz="0 0 1" />
+    <parent link="base_link"/>
+    <child link="right_back_wheel"/>
+    <origin rpy="0 ${M_PI/2} 0" xyz="${base_radius/cube_2} ${-base_radius/cube_2} -0.024"/>
+    <limit effort="100" velocity="100"/>
+    <joint_properties damping="0.0" friction="0.0"/>
+  </joint>
+  <joint name="left_front_wheel_joint" type="continuous">
+    <parent link="base_link"/>
+    <axis xyz="0 0 1" />
+    <child link="left_front_wheel"/>
+    <origin rpy="0 ${M_PI/2} 0" xyz="${-base_radius/cube_2} ${base_radius/cube_2} -0.024"/>
+    <limit effort="100" velocity="100"/>
+    <joint_properties damping="0.0" friction="0.0"/>
+  </joint>
+  <joint name="left_back_wheel_joint" type="continuous">
+    <parent link="base_link"/>
+    <axis xyz="0 0 1" />
+    <child link="left_back_wheel"/>
+    <origin rpy="0 ${M_PI/2} 0" xyz="${-base_radius/cube_2} ${-base_radius/cube_2} -0.024"/>
+    <limit effort="100" velocity="100"/>
+    <joint_properties damping="0.0" friction="0.0"/>
+  </joint>
   <!-- Drive controller -->
   <gazebo>
@@ -129,11 +106,14 @@
       <updateRate>100.0</updateRate>
       <robotNamespace></robotNamespace>
-      <leftFrontJoint>front_wheel</leftFrontJoint>
-      <rightFrontJoint>behind_left_wheel</rightFrontJoint>
-      <leftRearJoint>behind_right_wheel</leftRearJoint>
+      <leftFrontJoint>left_front_wheel_joint</leftFrontJoint>
+      <rightFrontJoint>right_front_wheel_joint</rightFrontJoint>
+      <leftRearJoint>left_back_wheel_joint</leftRearJoint>
+      <rightRearJoint>right_back_wheel_joint</rightRearJoint>
       <wheelSeparation>4</wheelSeparation>
       <wheelDiameter>0.1</wheelDiameter>
       <commandTopic>cmd_vel</commandTopic>
+      <odometryTopic>odom</odometryTopic>
       <robotBaseFrame>base_link</robotBaseFrame>
+      <odometryFrame>odom</odometryFrame>
       <torque>1</torque>
       <topicName>cmd_vel</topicName>

Commit message: 修改后的TMROBOT模型

File: test_gazebo_robot_model/urdf/my_move_robot.xacro (robot description, xacro)
@@ -22,5 +22,5 @@
 			</geometry>
 			<!-- <origin rpy="0 1.5 0" xyz="0.1 0.1 0"/> -->
-			<origin rpy="0 0 1.57075" xyz="0 0 0"/>
+			<origin rpy="0 0 ${M_PI/2}" xyz="0 0 0"/>
 			<material name="black">
 				<color rgba="0 0 0 1"/>
@@ -38,5 +38,5 @@
 				<cylinder length=".01" radius="${base_radius}"/>
 			</geometry>
-			<origin rpy="0 0 1.57075" xyz="0 0 0"/>
+			<origin rpy="0 0 ${M_PI/2}" xyz="0 0 0"/>
 			<material name="white">
 				<color rgba="1 1 1 1"/>
@@ -51,21 +51,21 @@
 	<link name="base_link">
 		<xacro:default_base_link />
-		<xacro:default_inertial mass="10"/>
+		<xacro:default_inertial mass="4"/>
 	</link>
 	<link name="right_front_wheel">
 		<xacro:default_wheel />
-		<xacro:default_inertial mass="0.01"/>
+		<xacro:default_inertial mass="1"/>
 	</link>
 	<link name="right_back_wheel">
 		<xacro:default_wheel />
-		<xacro:default_inertial mass="0.01"/>
+		<xacro:default_inertial mass="1"/>
 	</link>
 	<link name="left_front_wheel">
 		<xacro:default_wheel />
-		<xacro:default_inertial mass="0.01"/>
+		<xacro:default_inertial mass="1"/>
 	</link>
 	<link name="left_back_wheel">
 		<xacro:default_wheel />
-		<xacro:default_inertial mass="0.01"/>
+		<xacro:default_inertial mass="1"/>
 	</link>
 	<joint name="right_front_wheel_joint" type="continuous">
@@ -105,17 +105,17 @@
 	  <plugin name="skid_steer_drive_controller" filename="libgazebo_ros_skid_steer_drive.so">
 	    <updateRate>100.0</updateRate>
-	    <robotNamespace></robotNamespace>
+	    <robotNamespace>/</robotNamespace>
 	    <leftFrontJoint>left_front_wheel_joint</leftFrontJoint>
 	    <rightFrontJoint>right_front_wheel_joint</rightFrontJoint>
 	    <leftRearJoint>left_back_wheel_joint</leftRearJoint>
 	    <rightRearJoint>right_back_wheel_joint</rightRearJoint>
-	    <wheelSeparation>4</wheelSeparation>
-	    <wheelDiameter>0.1</wheelDiameter>
+	    <wheelSeparation>0.4</wheelSeparation>
+	    <wheelDiameter>0.215</wheelDiameter>
+	    <robotBaseFrame>base_link</robotBaseFrame>
+	    <torque>20</torque>
 	    <commandTopic>cmd_vel</commandTopic>
-	    <odometryTopic>odom</odometryTopic>
-	    <robotBaseFrame>base_link</robotBaseFrame>
-	    <odometryFrame>odom</odometryFrame>
-	    <torque>1</torque>
 	    <topicName>cmd_vel</topicName>
+		<odometryTopic>odom</odometryTopic>
+		<odometryFrame>odom</odometryFrame>
 	    <broadcastTF>1</broadcastTF>
 	  </plugin>
